File: DUT_Interface_board_v0.2.kicad_sch (KiCad schematic)
At the start: 193 parts, among them J1 USB1, J10 I2C_ext, J11 Frame_closure_switch, J12 Reed_Switch_servo, J13 Button_servo, J14 Conn_02x20_Odd_Even, J15 Conn_02x20_Odd_Even, J2 Power_profiler_interface, J20 digital_jumper_EE101, J22 AOUT, J25 shunt_jumper_EE101, J3 USB2, J4 Raspberry_Pi_2_3, J5 AD2_30_pin_connector, J6 Colour_sensor, J7 RF_Programmer, J8 SWD, J9 EE101, K1 UA2-5NJ_Relay_DPDT, Q1 AO3401A, Q2 TSM2302CX, Q3 TSM2302CX, Q4 TSM2302CX, Q5 TSM2302CX, Q6 TSM2302CX, U1 INA219AxDCN, U10 TXS0104EDR, U11 TXS0104EDR, U17 USBLC6-2SC6, U18 AMS1117, U3 USBLC6-2SC6, U4 ADS1015IDGS, U5 74HC4051, U6 74HC4051, U7 TXS0104EDR, U8 TXS0104EDR, U9 TXS0104EDR

Commit message: Math labels for inputs and outputs of U7.
Connections:
- net dig_1: now also U7.2 (A1); no longer U7.3 (A2)
- net dig_2: now also U7.3 (A2); no longer U7.4 (A3)
- net dig_3: now also U7.4 (A3); no longer U7.5 (A4)
- net dig_4: now also U7.5 (A4); no longer U7.2 (A1)
- net at JP56.2 (B): now also J15.1 (Pin_1); no longer J15.9 (Pin_9)
- net at JP31.2 (B): now also J15.9 (Pin_9); no longer J15.7 (Pin_7)
- net at J15.5 (Pin_5): no longer JP28.2 (B)
- net at J14.17 (Pin_17): now also JP73.2 (B)
- net at J14.19 (Pin_19): now also JP74.2 (B)
- net at J14.7 (Pin_7): no longer JP73.2 (B)
- net at J14.9 (Pin_9): no longer JP74.2 (B)
- new net: J15.7 (Pin_7), JP28.2 (B)
Other:
- note added: "TP1"
- note added: "TP10"
- note added: "TP13"
- note added: "TP14"
- note added: "TP15"
- note added: "TP18"
- note added: "TP19"
- note added: "TP2"
- note added: "TP20"
- note added: "TP21"
- note added: "TP22"
- note added: "TP23"
- note added: "TP24"
- note added: "TP25"
- note added: "TP26"
- note added: "TP27"
- note added: "TP28"
- note added: "TP29"
- note added: "TP3"
- note added: "TP30"
- note added: "TP34"
- note added: "TP35"
- note added: "TP36"
- note added: "TP4"
- note added: "TP6"
- note added: "TP7"
- note added: "TP9"
- moved on the sheet: J14, J15
